File: PTP_Josip_Bosnic_Project1.kicad_pcb (KiCad board)
At the start: 2 copper layers, 45 parts, among them J1 Screw_Terminal_01x02, SW1 SW_Push, SW2 SW_SPDT_312, U1 LM2574N-5, U2 4027, U3 4027, U4 74LS47, U5 HDSP-7401, U6 74LVC1G11, U7 NE555P

Commit message: v8
Parts:
- moved D5 27.5 mm to (178.2, 80.5), turned to 180 degrees
- moved R4 27.1 mm to (184.4, 80.5)
- moved R1 26.8 mm to (184.4, 104.2)
- moved R19 25.7 mm to (132.5, 106.0), turned to 180 degrees
- moved D1 24.6 mm to (178.0, 104.2), turned to 180 degrees
- moved U2 21.8 mm to (145.1, 86.8), turned to 0 degrees
- moved U3 17.0 mm to (159.4, 86.9), turned to 0 degrees
- moved C5 16.4 mm to (107.0, 92.0), turned to 180 degrees
- moved U6 16.3 mm to (157.8, 80.0)
- moved D4 14.1 mm to (141.8, 62.8), turned to 180 degrees
- moved R2 14.0 mm to (184.4, 96.0)
- moved D3 13.9 mm to (178.2, 88.5), turned to 180 degrees
- moved R3 13.7 mm to (184.4, 88.5)
- moved D2 11.8 mm to (178.2, 96.0), turned to 180 degrees
- moved R10 7.57 mm to (134.5, 93.0)
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Routing:
- net +5V: track 0.00 -> 261.8 mm, vias 0 -> 2
- net Q1: track 0.00 -> 97.9 mm, vias 0 -> 4
- net Q2: track 0.00 -> 72.3 mm, vias 0 -> 2
- net Q0: track 0.00 -> 64.4 mm
- net Q3: track 0.00 -> 52.5 mm, vias 0 -> 6
- net Clock: track 0.00 -> 48.8 mm, vias 0 -> 3
- net Reset: track 0.00 -> 45.6 mm, vias 0 -> 5
- net Net-(U4-BI): track 0.00 -> 43.0 mm
- net Net-(U2B-J): track 0.00 -> 40.4 mm
- net Net-(U7-DIS): track 0.00 -> 35.7 mm
- net Net-(U2A-J): track 0.00 -> 34.6 mm, vias 0 -> 2
- net Net-(U3A-J): track 0.00 -> 33.9 mm, vias 0 -> 2
- net Net-(U7-THR): track 0.00 -> 33.1 mm, vias 0 -> 2
- net Net-(U3B-J): track 0.00 -> 32.9 mm, vias 0 -> 2
- net Net-(SW2-A): track 0.00 -> 31.6 mm, vias 0 -> 2
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- added copper zone on B.Cu, net GND

Commit message: lab5
Routing:
- net GND: track 2.27 -> 20.7 mm, vias 0 -> 2
- net Q1: track 97.9 -> 99.9 mm, vias 4 -> 6
Other:
- board outline added: 100 x 80 mm
- board text added: "Josip Bosnić"
Changed lines of the file:
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@@
 			(usegerberattributes yes)
 			(usegerberadvancedattributes yes)
-			(creategerberjobfile yes)
+			(creategerberjobfile no)
 			(dashed_line_dash_ratio 12.000000)
 			(dashed_line_gap_ratio 3.000000)
@@
 			(outputformat 1)
 			(mirror no)
-			(drillshape 1)
+			(drillshape 0)
 			(scaleselection 1)
-			(outputdirectory "")
+			(outputdirectory "Manufacturing/")
 		)
 	)
@@
 		(stroke
 			(width 0.2)
-			(type default)
+			(type solid)
 		)
-		(layer "F.Cu")
+		(layer "Edge.Cuts")
 	)
 	(gr_line
@@
 		(stroke
 			(width 0.2)
-			(type default)
+			(type solid)
 		)
-		(layer "F.Cu")
+		(layer "Edge.Cuts")
 	)
 	(gr_arc
@@
 		(stroke
 			(width 0.2)
-			(type default)
+			(type solid)
 		)
-		(layer "F.Cu")
+		(layer "Edge.Cuts")
 	)
 	(gr_arc
@@
 		(stroke
 			(width 0.2)
-			(type default)
+			(type solid)
 		)
-		(layer "F.Cu")
+		(layer "Edge.Cuts")
 	)
 	(gr_line
@@
 		(stroke
 			(width 0.2)
-			(type default)
+			(type solid)
 		)
-		(layer "F.Cu")
+		(layer "Edge.Cuts")
 	)
 	(gr_line
@@
 		(stroke
 			(width 0.2)
-			(type default)
+			(type solid)
 		)
-		(layer "F.Cu")
+		(layer "Edge.Cuts")
 	)
 	(gr_arc
@@
 		(stroke
 			(width 0.2)
-			(type default)
+			(type solid)
 		)
-		(layer "F.Cu")
+		(layer "Edge.Cuts")
 	)
 	(gr_line
@@
 		(stroke
 			(width 0.2)
-			(type default)
+			(type solid)
 		)
+		(layer "Edge.Cuts")
+	)
+	(gr_text "Josip Bosnić"
+		(at 168 118 0)
+		(layer "F.SilkS")
+		(effects
+			(font
+				(size 1 1)
+				(thickness 0.1)
+			)
+			(justify left bottom)
+		)
+	)
+	(segment
+		(start 157.037678 80)
+		(end 157.874 79.163678)
+		(width 0.3)
 		(layer "F.Cu")
+		(net 1)
 	)
 	(segment
@@
 	)
 	(segment
+		(start 117.875 77)
+		(end 113.5 77)
+		(width 0.2)
+		(layer "F.Cu")
+		(net 1)
+	)
+	(segment
+		(start 157.874 79.163678)
+		(end 157.874 78.626)
+		(width 0.3)
+		(layer "F.Cu")
+		(net 1)
+	)
+	(segment
+		(start 156.6125 80)
+		(end 157.037678 80)
+		(width 0.3)
+		(layer "F.Cu")
+		(net 1)
+	)
+	(segment
 		(start 194.58 104.25)
 		(end 194.58 105.67)
@@
 	)
 	(segment
+		(start 113.5 77)
+		(end 111.5 79)
+		(width 0.2)
+		(layer "F.Cu")
+		(net 1)
+	)
+	(segment
+		(start 157.874 78.626)
+		(end 158.5 78)
+		(width 0.3)
+		(layer "F.Cu")
+		(net 1)
+	)
+	(segment
 		(start 124.69 56.31)
 		(end 124.69 55.81)
@@
 	)
 	(segment
+		(start 105.4375 92)
+		(end 105.4375 98.5)
+		(width 0.2)
+		(layer "F.Cu")
+		(net 1)
+	)
+	(segment
+		(start 158.5 78)
+		(end 159 78)
+		(width 0.3)
+		(layer "F.Cu")
+		(net 1)
+	)
+	(via
+		(at 159 78)
+		(size 0.7)
+		(drill 0.3)
+		(layers "F.Cu" "B.Cu")
+		(net 1)
+	)
+	(via
+		(at 105.4375 95.5)
+		(size 0.7)
+		(drill 0.3)
+		(layers "F.Cu" "B.Cu")
+		(net 1)
+	)
+	(segment
+		(start 155.69 66.89)
+		(end 156.5 67.7)
+		(width 0.2)
+		(layer "B.Cu")
+		(net 1)
+	)
+	(segment
 		(start 119.101 62.101)
 		(end 123.649 62.101)
@@
 	)
 	(segment
+		(start 158.8875 79.05)
+		(end 160.45 79.05)
+		(width 0.3)
+		(layer "F.Cu")
+		(net 9)
+	)
+	(segment
 		(start 151.75 49)
 		(end 151.86 49.11)
@@
 	)
 	(segment
-		(start 175.291 95.581)
-		(end 163.081 95.581)
-		(width 0.2)
+		(start 160.45 79.05)
+		(end 160.5 79)
+		(width 0.3)
 		(layer "F.Cu")
 		(net 9)
 	)
 	(segment
-		(start 157.924 79.351001)
-		(end 158.225001 79.05)
+		(start 175.291 95.581)
+		(end 163.081 95.581)
 		(width 0.2)
 		(layer "F.Cu")
@@
 	)
 	(segment
-		(start 158.225001 79.05)
-		(end 158.8875 79.05)
-		(width 0.2)
-		(layer "F.Cu")
-		(net 9)
-	)
-	(segment
-		(start 157.924 84.166)
-		(end 157.924 79.351001)
-		(width 0.2)
-		(layer "F.Cu")
-		(net 9)
-	)
-	(segment
 		(start 159.44 91.94)
 		(end 155.35 91.94)
@@
 	)
 	(via
+		(at 160.5 79)
+		(size 0.7)
+		(drill 0.3)
+		(layers "F.Cu" "B.Cu")
+		(net 9)
+	)
+	(via
+		(at 157.924 84.166)
+		(size 0.7)
+		(drill 0.3)
+		(layers "F.Cu" "B.Cu")
+		(net 9)
+	)
+	(via
 		(at 155.75 88.25)
 		(size 0.7)
@@
 	)
 	(segment
+		(start 160.5 79)
+		(end 160.5 81.741364)
+		(width 0.3)
+		(layer "B.Cu")
+		(net 9)
+	)
+	(segment
 		(start 155.75 83)
 		(end 141.25 68.5)
@@
 		(layer "B.Cu")
 		(net 9)
+	)
+	(segment
+		(start 160.5 81.741364)
+		(end 158.075364 84.166)
+		(width 0.3)
+		(layer "B.Cu")
+		(net 9)
+	)
+	(segment
+		(start 158.075364 84.166)
+		(end 157.924 84.166)
+		(width 0.3)
+		(layer "B.Cu")
+		(net 9)
